File: KiCad/bga_0201_rect/bga_0201_rect.kicad_pcb (KiCad board)
At the start: 4 copper layers, 6 x 24.7 mm, 15 parts, among them J1 JST-ZH, J2 Conn_ARM_SWD_TagConnect_TC203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, U1 NCP163AFCS120T2G, U2 STM32C011D6Yx, U4 LIS2DE12, Y1 ASE-xxxMHz

Commit message: updated bga_0201_rect
Parts:
- Y1: footprint Oscillator:Oscillator_SMD_Abracon_ASE-4Pin_3.2x2.5mm -> Crystal:Crystal_SMD_EuroQuartz_MT-4Pin_3.2x2.5mm
Changed lines of the file:
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@@
 			(plot_on_all_layers_selection 0x00000000_00000000_00000000_00000000)
 			(disableapertmacros no)
-			(usegerberextensions yes)
+			(usegerberextensions no)
 			(usegerberattributes yes)
 			(usegerberadvancedattributes yes)
@@
 			(drillshape 0)
 			(scaleselection 1)
-			(outputdirectory "ouputs/gbr_protel/")
+			(outputdirectory "assets/gbr_default/")
 		)
 	)
@@
 		)
 		(embedded_fonts no)
-		(model "${KICAD9_3DMODEL_DIR}/Package_CSP.3dshapes/ST_WLCSP-12_1.7x1.42mm_Layout4x6_P0.35mm_Stagger.step"
+		(model "${KIPRJMOD}/WLCSP12_1P7X1P42_STM.step"
 			(offset
 				(xyz 0 0 0)
@@
 		)
 		(embedded_fonts no)
-		(model "${KICAD9_3DMODEL_DIR}/Connector_JST.3dshapes/JST_ZH_B2B-ZR_1x02_P1.50mm_Vertical.step"
+		(model "${KIPRJMOD}/B2B-ZR.step"
 			(offset
 				(xyz 0 0 0)
@@
 			)
 			(rotate
-				(xyz 0 0 0)
+				(xyz -0 -0 90)
 			)
 		)
@@
 		)
 	)
-	(footprint "Oscillator:Oscillator_SMD_Abracon_ASE-4Pin_3.2x2.5mm"
+	(footprint "Crystal:Crystal_SMD_EuroQuartz_MT-4Pin_3.2x2.5mm"
 		(layer "F.Cu")
 		(at 33.3 35.6)
-		(descr "Abracon ASE, Miniature Crystal Clock Oscillator, 3.2x2.5mm package, SMD, generated with kicad-footprint-generator make_crystal.py, http://www.abracon.com/Oscillators/ASEseries.pdf")
-		(tags "SMD SMT crystal oscillator")
+		(descr "EuroQuartz MT, Crystal, 3.2x2.5mm package, SMD, generated with kicad-footprint-generator make_crystal.py, http://cdn-reichelt.de/documents/datenblatt/B400/MT.pdf")
 		(property "Reference" "Y1"
 			(at 0 -2.45 0)
@@
 			(at 0 2.45 0)
 			(layer "F.Fab")
-			(hide yes)
 			(effects
 				(font
@@
 		(attr smd)
 		(fp_line
-			(start -1.96 -1.635)
-			(end -1.96 1.635)
+			(start -2.01 -1.66)
+			(end -2.01 1.66)
 			(stroke
 				(width 0.12)
@@
 		)
 		(fp_line
-			(start -1.96 1.635)
-			(end 1.96 1.635)
+			(start -2.01 1.66)
+			(end 2.01 1.66)
 			(stroke
 				(width 0.12)
@@
 			(layer "F.SilkS")
 		)
-		(fp_circle
-			(center 0 0)
-			(end 0.25 0)
-			(stroke
-				(width 0.1)
-				(type solid)
-			)
-			(fill yes)
-			(layer "F.Adhes")
-		)
 		(fp_rect
 			(start -2.1 -1.75)
@@
 			(layer "F.Fab")
 		)
+		(fp_text user "${REFERENCE}"
+			(at 0 0 0)
+			(layer "F.Fab")
+			(effects
+				(font
+					(size 0.8 0.8)
+					(thickness 0.12)
+				)
+			)
+		)
 		(pad "1" smd roundrect
-			(at -1.05 0.825)
-			(size 1.3 1.1)
+			(at -1.1 0.9)
+			(size 1.3 1)
 			(layers "F.Cu" "F.Mask" "F.Paste")
-			(roundrect_rratio 0.227273)
+			(roundrect_rratio 0.25)
 			(net 2 "VDD")
 			(pinfunction "EN")
@@
 		)
 		(pad "2" smd roundrect
-			(at 1.05 0.825)
-			(size 1.3 1.1)
+			(at 1.1 0.9)
+			(size 1.3 1)
 			(layers "F.Cu" "F.Mask" "F.Paste")
-			(roundrect_rratio 0.227273)
+			(roundrect_rratio 0.25)
 			(net 1 "GND")
 			(pinfunction "GND")
@@
 		)
 		(pad "3" smd roundrect
-			(at 1.05 -0.825)
-			(size 1.3 1.1)
+			(at 1.1 -0.9)
+			(size 1.3 1)
 			(layers "F.Cu" "F.Mask" "F.Paste")
-			(roundrect_rratio 0.227273)
+			(roundrect_rratio 0.25)
 			(net 14 "Net-(U2-PC14)")
 			(pinfunction "OUT")
@@
 		)
 		(pad "4" smd roundrect
-			(at -1.05 -0.825)
-			(size 1.3 1.1)
+			(at -1.1 -0.9)
+			(size 1.3 1)
 			(layers "F.Cu" "F.Mask" "F.Paste")
-			(roundrect_rratio 0.227273)
+			(roundrect_rratio 0.25)
 			(net 2 "VDD")
 			(pinfunction "Vdd")
@@
 		)
 		(embedded_fonts no)
-		(model "${KICAD9_3DMODEL_DIR}/Oscillator.3dshapes/Oscillator_SMD_Abracon_ASE-4Pin_3.2x2.5mm.step"
+		(model "${KICAD9_3DMODEL_DIR}/Crystal.3dshapes/Crystal_SMD_EuroQuartz_MT-4Pin_3.2x2.5mm.step"
 			(offset
 				(xyz 0 0 0)
@@
 		)
 		(embedded_fonts no)
-		(model "${KICAD9_3DMODEL_DIR}/Package_CSP.3dshapes/WLCSP-4_0.64x0.64mm_Layout2x2_P0.35mm.step"
+		(model "${KIPRJMOD}/WLCSP4_P7XP7_ONS.step"
 			(offset
 				(xyz 0 0 0)
@@
 		(net 3)
 	)
+	(segment
+		(start 32.9 41.2)
+		(end 33.114645 41.2)
+		(width 0.1)
+		(layer "F.Cu")
+		(net 3)
+	)
 	(via
 		(at 34.7 41.92)
@@
 	)
 	(arc
+		(start 33.114645 41.2)
+		(mid 33.147309 41.193502)
+		(end 33.175 41.175)
+		(width 0.1)
+		(layer "F.Cu")
+		(net 3)
+	)
+	(arc
 		(start 33.368457 41.368457)
 		(mid 33.979374 41.776658)
@@
 	)
 	(segment
-		(start 34.7 33.089949)
-		(end 34.7 33.358579)
-		(width 0.1)
-		(layer "F.Cu")
-		(net 14)
-	)
-	(segment
-		(start 34.35 34.203553)
-		(end 34.35 34.775)
+		(start 34.6 32.848528)
+		(end 34.6 34.217157)
 		(width 0.1)
 		(layer "F.Cu")
@@
 	)
 	(arc
-		(start 34.7 33.358579)
-		(mid 34.67401 33.489235)
-		(end 34.6 33.6)
-		(width 0.1)
-		(layer "F.Cu")
-		(net 14)
-	)
-	(arc
-		(start 34.6 33.6)
-		(mid 34.414973 33.876912)
-		(end 34.35 34.203553)
+		(start 33.400198 31.151554)
+		(mid 33.724808 31.216123)
+		(end 34 31.4)
 		(width 0.1)
 		(layer "F.Cu")
@@
 	(arc
 		(start 34 31.4)
-		(mid 34.518076 32.175355)
-		(end 34.7 33.089949)
+		(mid 34.444065 32.06459)
+		(end 34.6 32.848528)
 		(width 0.1)
 		(layer "F.Cu")
@@
 	)
 	(arc
-		(start 33.400198 31.151554)
-		(mid 33.724808 31.216123)
-		(end 34 31.4)
+		(start 34.6 34.217157)
+		(mid 34.548022 34.47847)
+		(end 34.4 34.7)
 		(width 0.1)
 		(layer "F.Cu")
