File: KiCad/bga_0201_rect/bga_0201_rect.kicad_sch (KiCad schematic)
At the start: 15 parts, among them J1 JST-ZH, J2 Conn_ARM_SWD_TagConnect_TC203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, U1 NCP163AFCS120T2G, U2 STM32C011D6Yx, U4 LIS2DE12, Y1 ASE-xxxMHz

Commit message: updated bga_0201_rect
Parts:
- Y1: footprint Oscillator:Oscillator_SMD_Abracon_ASE-4Pin_3.2x2.5mm -> Crystal:Crystal_SMD_EuroQuartz_MT-4Pin_3.2x2.5mm
Changed lines of the file:
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@@
 			)
 		)
-		(property "Footprint" "Oscillator:Oscillator_SMD_Abracon_ASE-4Pin_3.2x2.5mm"
+		(property "Footprint" "Crystal:Crystal_SMD_EuroQuartz_MT-4Pin_3.2x2.5mm"
 			(at 97.79 115.57 0)
 			(effects
